Commit message: 2024/12/3

File: urdf/lexus.urdf (robot description, URDF)
Before this commit: robot car, 1 links, 0 joints
Links:
- added link GPS
- added link laser_link
Joints:
- added joint GPS_joint: type fixed, parent base_link, child GPS, origin xyz=0 -3.995 0 rpy=0 0 1.570796327
- added joint laser_link_joint: type fixed, parent base_link, child laser_link, origin xyz=0 0 0 rpy=0 0 0
